File: hardware/filter_board/filter_board.kicad_pcb (KiCad board)
At the start: 2 copper layers, 100 x 60 mm, 47 parts, among them J101 Amphenol 031-6576, J102 Amphenol 031-6576, SW101 Grayhill 34ADP12B4M7GT

Commit message: Syncronizing with hardware files.
Connections:
- net Net-(C101-Pad2) renamed /Lbupper
- net Net-(C102-Pad2) renamed /Lbetween
- net Net-(C103-Pad2) renamed /Llower
- net Net-(C115-Pad2) renamed /Rbupper
- net Net-(C116-Pad2) renamed /Rbetween
- net Net-(C117-Pad2) renamed /Rlower
Routing:
- net /Lbupper: track 38.5 -> 41.7 mm
- added copper zone on F.Cu, net /Lbetween
- added copper zone on F.Cu, net /Lbupper
- added copper zone on F.Cu, net /Llower
- added copper zone on F.Cu, net /Rbetween
- added copper zone on F.Cu, net /Rbupper
- added copper zone on F.Cu, net /Rlower
