File: hardware/filter_board/filter_board.kicad_sch (KiCad schematic)
At the start: 47 parts, among them J101 Amphenol 031-6576, J102 Amphenol 031-6576, SW101 Grayhill 34ADP12B4M7GT

Commit message: Syncronizing with hardware files.
Connections:
- net Lbetween: now reaches C102.2, C103.1, C106.2, C107.1, C110.2, C111.1, C114.2, R101.2, R102.1, R106.2, R107.1
- net Lbupper: now reaches C101.2, C102.1, C105.2, C106.1, C109.2, C110.1, C113.2, C114.1
- net Rbupper: now reaches C115.2, C116.1, C119.2, C120.1, C123.2, C124.1, C127.2, C128.1
- net Rbetween: now reaches C116.2, C117.1, C120.2, C121.1, C124.2, C125.1, C128.2, R109.2, R110.1, R114.2, R115.1
- net Rlower: now reaches C117.2, C118.1, C121.2, C122.1, C125.2, C126.1
- net Llower: now reaches C103.2, C104.1, C107.2, C108.1, C111.2, C112.1
Other:
- company: (none) -> Erik Ø. Sørensen, LB3TH
- title: (none) -> Inverse RIAA filter
Changed lines of the file:
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@@
 (kicad_sch (version 20230121) (generator eeschema)
   (paper "A4")
+  (title_block
+    (title "Inverse RIAA filter")
+    (date "2023-12-10")
+    (company "Erik Ø. Sørensen, LB3TH")
+  )
   (junction (at 215.9 99.06) (diameter 0) (color 0 0 0 0)
   )
@@
     (stroke (width 0) (type default))
   )
+  (label "Llower" (at 100.33 86.36 0) (fields_autoplaced)
+    (effects (font (size 1.27 1.27)) (justify left bottom))
+  )
+  (label "Rbupper" (at 205.74 53.34 0) (fields_autoplaced)
+    (effects (font (size 1.27 1.27)) (justify left bottom))
+  )
+  (label "Rlower" (at 208.28 86.36 0) (fields_autoplaced)
+    (effects (font (size 1.27 1.27)) (justify left bottom))
+  )
+  (label "Lbetween" (at 83.82 69.85 0) (fields_autoplaced)
+    (effects (font (size 1.27 1.27)) (justify left bottom))
+  )
+  (label "Lbupper" (at 99.06 53.34 0) (fields_autoplaced)
+    (effects (font (size 1.27 1.27)) (justify left bottom))
+  )
+  (label "Rbetween" (at 193.04 69.85 0) (fields_autoplaced)
+    (effects (font (size 1.27 1.27)) (justify left bottom))
+  )
   (global_label "Lmm" (shape input) (at 96.52 104.14 0) (fields_autoplaced)
